File: ethernet.kicad_sch (KiCad schematic)
At the start: 22 parts, among them J2 L834-1G1T-S7, Q2 PMOS_Substrate, U2 LAN8830T_PSA

Commit message: Import all symbols into project library
Parts:
- J2: symbol snapmaker-footprints:L834-1G1T-S7 -> Library:L834-1G1T-S7
- U2: symbol LAN8830T_PSA:LAN8830T_PSA -> Library:LAN8830T_PSA
Changed lines of the file:
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@@
 	)
 	(symbol
-		(lib_id "snapmaker-footprints:L834-1G1T-S7")
+		(lib_id "Library:L834-1G1T-S7")
 		(at 194.31 105.41 0)
 		(unit 1)
@@
 		(exclude_from_sim no)
 		(in_bom yes)
-		(on_board no)
+		(on_board yes)
 		(in_pos_files yes)
 		(dnp no)
@@
 		)
 		(property "Footprint" "L834-1G1T-S7:BEL_L834-1G1T-S7"
-			(at 194.31 105.41 0)
+			(at 161.798 131.318 0)
 			(hide yes)
 			(show_name no)
@@
 		)
 		(property "Datasheet" ""
-			(at 194.31 105.41 0)
+			(at 154.94 105.41 0)
 			(hide yes)
 			(show_name no)
@@
 		)
 		(property "Description" "MagJack 1000BASE-T | 1X1 | G/G | Tab Down | Low Profile | RoHS"
-			(at 194.31 105.41 0)
+			(at 148.082 112.522 0)
 			(hide yes)
 			(show_name no)
@@
 		)
 		(property "MF" "Bel Fuse Inc."
-			(at 194.31 105.41 0)
+			(at 194.564 147.32 0)
 			(hide yes)
 			(show_name no)
@@
 		)
 		(property "PACKAGE" "None"
-			(at 194.31 105.41 0)
+			(at 154.94 105.41 0)
 			(hide yes)
 			(show_name no)
@@
 		)
 		(property "PRICE" "None"
-			(at 194.31 105.41 0)
+			(at 154.94 105.41 0)
 			(hide yes)
 			(show_name no)
@@
 		)
 		(property "Package" "None"
-			(at 194.31 105.41 0)
+			(at 154.94 105.41 0)
 			(hide yes)
 			(show_name no)
@@
 		)
 		(property "Check_prices" "https://www.snapeda.com/parts/L834-1G1T-S7/Bel+Circuit+Protection/view-part/?ref=eda"
-			(at 194.31 105.41 0)
+			(at 194.564 152.146 0)
 			(hide yes)
 			(show_name no)
@@
 		)
 		(property "Price" "None"
-			(at 194.31 105.41 0)
+			(at 154.94 105.41 0)
 			(hide yes)
 			(show_name no)
@@
 		)
 		(property "SnapEDA_Link" "https://www.snapeda.com/parts/L834-1G1T-S7/Bel+Circuit+Protection/view-part/?ref=snap"
-			(at 194.31 105.41 0)
+			(at 142.494 117.094 0)
 			(hide yes)
 			(show_name no)
@@
 		)
 		(property "MP" "L834-1G1T-S7"
-			(at 194.31 105.41 0)
+			(at 150.368 114.046 0)
 			(hide yes)
 			(show_name no)
@@
 		)
 		(property "DIGIKEY-PURCHASE-URL" "https://snapeda.com/shop?store=DigiKey&id=4797102"
-			(at 194.31 105.41 0)
+			(at 194.31 144.78 0)
 			(hide yes)
 			(show_name no)
@@
 		)
 		(property "Availability" "In Stock"
-			(at 194.31 105.41 0)
+			(at 154.686 112.522 0)
 			(hide yes)
 			(show_name no)
@@
 		)
 		(property "AVAILABILITY" "Unavailable"
-			(at 194.31 105.41 0)
+			(at 145.288 99.06 0)
 			(hide yes)
 			(show_name no)
@@
 	)
 	(symbol
-		(lib_id "LAN8830T_PSA:LAN8830T_PSA")
+		(lib_id "Library:LAN8830T_PSA")
 		(at 113.03 99.06 0)
 		(unit 1)
@@
 		(exclude_from_sim no)
 		(in_bom yes)
-		(on_board no)
+		(on_board yes)
 		(in_pos_files yes)
 		(dnp no)
@@
 		)
 		(property "Footprint" "LAN8830T_PSA:QFN50P700X700X100-49N"
+			(at 105.41 99.06 0)
+			(hide yes)
+			(show_name no)
+			(do_not_autoplace no)
+			(effects
+				(font
+					(size 1.27 1.27)
+				)
+				(justify bottom)
+			)
+		)
+		(property "Datasheet" ""
 			(at 113.03 99.06 0)
 			(hide yes)
@@
 					(size 1.27 1.27)
 				)
+			)
+		)
+		(property "Description" "4/4 Transceiver Full, Half Ethernet 48-VQFN (7x7)"
+			(at 105.41 99.06 0)
+			(hide yes)
+			(show_name no)
+			(do_not_autoplace no)
+			(effects
+				(font
+					(size 1.27 1.27)
+				)
 				(justify bottom)
 			)
 		)
-		(property "Datasheet" ""
-			(at 113.03 99.06 0)
-			(hide yes)
-			(show_name no)
-			(do_not_autoplace no)
-			(effects
-				(font
-					(size 1.27 1.27)
-				)
-			)
-		)
-		(property "Description" "4/4 Transceiver Full, Half Ethernet 48-VQFN (7x7)"
-			(at 113.03 99.06 0)
+		(property "DigiKey_Part_Number" "150-LAN8830T/PSACT-ND"
+			(at 105.41 99.06 0)
 			(hide yes)
 			(show_name no)
@@
 			)
 		)
-		(property "DigiKey_Part_Number" "150-LAN8830T/PSACT-ND"
-			(at 113.03 99.06 0)
+		(property "SnapEDA_Link" "https://www.snapeda.com/parts/LAN8830T/PSA/Microchip+Technology/view-part/?ref=snap"
+			(at 105.41 99.06 0)
 			(hide yes)
 			(show_name no)
@@
 			)
 		)
-		(property "SnapEDA_Link" "https://www.snapeda.com/parts/LAN8830T/PSA/Microchip+Technology/view-part/?ref=snap"
-			(at 113.03 99.06 0)
+		(property "MAXIMUM_PACKAGE_HEIGHT" "1mm"
+			(at 105.41 99.06 0)
 			(hide yes)
 			(show_name no)
@@
 			)
 		)
-		(property "MAXIMUM_PACKAGE_HEIGHT" "1mm"
-			(at 113.03 99.06 0)
+		(property "Package" "None"
+			(at 105.41 99.06 0)
 			(hide yes)
 			(show_name no)
@@
 			)
 		)
-		(property "Package" "None"
-			(at 113.03 99.06 0)
+		(property "Check_prices" "https://www.snapeda.com/parts/LAN8830T/PSA/Microchip+Technology/view-part/?ref=eda"
+			(at 105.41 99.06 0)
 			(hide yes)
 			(show_name no)
@@
 			)
 		)
-		(property "Check_prices" "https://www.snapeda.com/parts/LAN8830T/PSA/Microchip+Technology/view-part/?ref=eda"
-			(at 113.03 99.06 0)
+		(property "STANDARD" "Manufacturer Recommendations"
+			(at 105.41 99.06 0)
 			(hide yes)
 			(show_name no)
@@
 			)
 		)
-		(property "STANDARD" "Manufacturer Recommendations"
-			(at 113.03 99.06 0)
+		(property "PARTREV" "DS00004724A"
+			(at 105.41 99.06 0)
 			(hide yes)
 			(show_name no)
@@
 			)
 		)
-		(property "PARTREV" "DS00004724A"
-			(at 113.03 99.06 0)
+		(property "MF" "Microchip Technology"
+			(at 105.41 99.06 0)
 			(hide yes)
 			(show_name no)
@@
 			)
 		)
-		(property "MF" "Microchip Technology"
-			(at 113.03 99.06 0)
+		(property "MP" "LAN8830T/PSA"
+			(at 105.41 99.06 0)
 			(hide yes)
 			(show_name no)
@@
 			)
 		)
-		(property "MP" "LAN8830T/PSA"
-			(at 113.03 99.06 0)
+		(property "SNAPEDA_PN" "LAN8830/PSA"
+			(at 105.41 99.06 0)
 			(hide yes)
 			(show_name no)
@@
 			)
 		)
-		(property "SNAPEDA_PN" "LAN8830/PSA"
-			(at 113.03 99.06 0)
-			(hide yes)
-			(show_name no)
-			(do_not_autoplace no)
-			(effects
-				(font
-					(size 1.27 1.27)
-				)
-				(justify bottom)
-			)
-		)
 		(property "MANUFACTURER" "Microchip"
-			(at 113.03 99.06 0)
-			(hide yes)
-			(show_name no)
+			(at 105.41 99.06 0)
+			(hide yes)
+			(show_name no)
