File: little-witch.kicad_sch (KiCad schematic)
At the start: 32 parts, among them J1 GCT-USB4105, J3 Conn_ARM_SWD_TagConnect_TC203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, J4 GCT-USB4105, J5 Conn_02x20_Odd_Even, SW1 RESET, SW2 BOOT0, U1 CH32V307RCT6, Y1 SIT8008BI-73-33N-25.000000

Commit message: Start of USB changes
Parts:
- removed JP5: SolderJumper_2_Open, Jumper:SolderJumper-2_P1.3mm_Open_RoundedPad1.0x1.5mm, symbol Jumper:SolderJumper_2_Open
- added D2: D_Schottky, symbol Device:D_Schottky
- added R25: 10k, Resistor_SMD:R_0402_1005Metric, symbol Device:R_Small_US
- added SW3: SW_SPST, symbol Switch:SW_SPST
- R10: value 10k -> 100k
Connections:
- net VBUS: now also SW3.2 (B)
- net at J1.A4 (VBUS), J1.A9 (VBUS), J1.B4 (VBUS)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: now also D2.1 (K); no longer D1.2 (A)
- net at R10.2, SW2.2, U1.60 (BOOT0): now also R25.2; no longer C14.2
- net at J4.A4 (VBUS), J4.A9 (VBUS), J4.B4 (VBUS)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: now also D1.2 (A)
- new net: C14.2, R25.1
- new net USB2_VBUS: D2.2 (A), SW3.1 (A)
- no-connect marks 6 -> 5
